File: IR_Station/eagle v2.0/SolderingStation.brd (EAGLE design)
At the start: 160 x 100 mm, 112 parts, among them IC1 LM317, U1 MSP340G2443, U2 UPD166010, U3 MCP6V08, U4 UPD166010, U5 MCP6V08, U6 ADS1115IDGST

Commit message: 04.04.2018
Connections:
- net 220V_DRIVER_UC: now also JP6.1, U1.5; no longer JP9.3, U1.21
- net DATA_DISPLAY: now also JP9.3, U1.21; no longer JP6.1, U1.5
Routing:
- net DATA_DISPLAY: track 9.55 -> 18.9 mm
- net 220V_DRIVER_UC: track 18.9 -> 9.55 mm
Changed lines of the file:
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@@
 <wire x1="116.81" y1="60.5" x2="114.5" y2="60.5" width="0.8128" layer="1"/>
-</signal>
-<signal name="DATA_DISPLAY">
-<contactref element="U1" pad="5"/>
-<wire x1="60.77" y1="24.27" x2="61.5" y2="25" width="0.3048" layer="1"/>
-<wire x1="65.65365" y1="28.872" x2="65.65365" y2="26.40365" width="0.3048" layer="1"/>
-<wire x1="65.65365" y1="26.40365" x2="64.25" y2="25" width="0.3048" layer="1"/>
-<wire x1="64.25" y1="25" x2="61.5" y2="25" width="0.3048" layer="1"/>
-<contactref element="JP6" pad="1"/>
-<wire x1="60.81" y1="23" x2="60.77" y2="23" width="0.4064" layer="1"/>
-<wire x1="60.77" y1="23" x2="60.77" y2="24.27" width="0.4064" layer="1"/>
 </signal>
 <signal name="TEST">
@@
 </signal>
 <signal name="220V_DRIVER_UC">
-<contactref element="U1" pad="21"/>
-<contactref element="JP9" pad="3"/>
-<wire x1="67.60365" y1="34.6721" x2="67.60365" y2="39.35365" width="0.3048" layer="1"/>
-<wire x1="67.60365" y1="39.35365" x2="70.5" y2="42.25" width="0.3048" layer="1"/>
-<wire x1="70.5" y1="42.25" x2="77" y2="42.25" width="0.3048" layer="1"/>
-<wire x1="77" y1="42.25" x2="78" y2="43.25" width="0.3048" layer="1"/>
-<wire x1="78" y1="43.25" x2="78" y2="44.17" width="0.3048" layer="1"/>
-<wire x1="78" y1="44.17" x2="77.92" y2="45.5" width="0.3048" layer="1"/>
+<contactref element="U1" pad="5"/>
+<wire x1="60.77" y1="24.27" x2="61.5" y2="25" width="0.3048" layer="1"/>
+<wire x1="65.65365" y1="28.872" x2="65.65365" y2="26.40365" width="0.3048" layer="1"/>
+<wire x1="65.65365" y1="26.40365" x2="64.25" y2="25" width="0.3048" layer="1"/>
+<wire x1="64.25" y1="25" x2="61.5" y2="25" width="0.3048" layer="1"/>
+<contactref element="JP6" pad="1"/>
+<wire x1="60.81" y1="23" x2="60.77" y2="23" width="0.4064" layer="1"/>
+<wire x1="60.77" y1="23" x2="60.77" y2="24.27" width="0.4064" layer="1"/>
 </signal>
 <signal name="LATCH_DISPLAY">
@@
 <wire x1="85" y1="26" x2="85" y2="22.75" width="1.016" layer="1"/>
 </signal>
+<signal name="DATA_DISPLAY">
+<contactref element="U1" pad="21"/>
+<contactref element="JP9" pad="3"/>
+<wire x1="67.60365" y1="34.6721" x2="67.60365" y2="39.35365" width="0.3048" layer="1"/>
+<wire x1="67.60365" y1="39.35365" x2="70.5" y2="42.25" width="0.3048" layer="1"/>
+<wire x1="70.5" y1="42.25" x2="77" y2="42.25" width="0.3048" layer="1"/>
+<wire x1="77" y1="42.25" x2="78" y2="43.25" width="0.3048" layer="1"/>
+<wire x1="78" y1="43.25" x2="78" y2="44.17" width="0.3048" layer="1"/>
+<wire x1="78" y1="44.17" x2="77.92" y2="45.5" width="0.3048" layer="1"/>
+</signal>
 </signals>
