File: IR_Station/eagle v2.0/SolderingStation.sch (EAGLE design)
At the start: 104 parts, among them IC1 LM317, J1 JP4, J2 JP4, J3 JP4, J4 JP4, U1 MSP340G2443, U2 UPD166010, U3 MCP6V08, U4 UPD166010, U5 MCP6V08, U6 ADS1115IDGST

Commit message: Update linse from all pins! some features :)
Parts:
- added C15, C8: 1nF, adi_v1.2:C0805
- added JP11: (no value), pinhead:PINHD-1X2
- added JP15: (no value), pinhead:PINHD-1X1
- added JP16: (no value), pinhead:PINHD-1X5
- added R25: 87R, adi_v1.2:R0805
- added R34: 0R, adi_v1.2:R0805
- added U$12: (no value), Serghei IR station:COIL
- JP1: device pinhead:PINHD-1X4/90 -> pinhead:PINHD-1X2
- JP6: device pinhead:PINHD-1X6 -> pinhead:PINHD-1X4
Connections:
- new net N$2222: JP1.1, LED1.A
- new net N$37: C8.1, U$12.P$2, U1.6
- new net N$39: C15.1, U$12.P$1, U1.7
- new net N$45: JP15.1, R25.1
- new net N$46: CLH1.IN, R34.1
- net +3V3_220V: now also JP16.2; no longer JP1.1
- net 24V_CS_UC: now also JP6.4; no longer JP6.6
- net 24V_PWM: now also R25.2, R34.2; no longer CLH1.IN
- net DATA_DISPLAY: now also JP6.1; no longer JP6.3
- net GND_220V: now also JP16.5; no longer JP1.4
- net GND_UC: now also C15.2, C8.2
- net N$15: now also JP16.4; no longer JP1.3
- net N$17: now also JP1.2, JP16.1; no longer LED1.A
- net N$36: now also JP16.3; no longer JP1.2
- net RX: now also JP6.3; no longer JP6.5
- net TIP_TEMP1_UC: now also JP11.2, U$12.P$3; no longer JP6.2, U1.6
- net TIP_TEMP2_UC: now also JP11.1, U$12.P$4; no longer JP6.1, U1.7
- net TX: now also JP6.2; no longer JP6.4
Other:
- note added: "15mA"
- moved on the sheet: LED1

Commit message: 04.04.2018
Connections:
- net 220V_DRIVER_UC: now also JP6.1, U1.5; no longer JP9.3, U1.21
- net DATA_DISPLAY: now also JP9.3, U1.21; no longer JP6.1, U1.5
Changed lines of the file:
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@@
-</segment>
-</net>
-<net name="DATA_DISPLAY" class="0">
-<segment>
-<pinref part="U1" gate="G$1" pin="5"/>
-<label x="176.53" y="48.514" size="1.27" layer="95" rot="R180" xref="yes"/>
-<wire x1="179.07" y1="48.514" x2="150.876" y2="48.514" width="0.1524" layer="91"/>
-<pinref part="JP6" gate="A" pin="1"/>
 </segment>
 </net>
@@
 <net name="220V_DRIVER_UC" class="0">
 <segment>
-<pinref part="U1" gate="G$1" pin="21"/>
-<label x="229.87" y="40.894" size="1.27" layer="95" xref="yes"/>
-<wire x1="226.06" y1="40.894" x2="254" y2="40.894" width="0.1524" layer="91"/>
-<pinref part="JP9" gate="A" pin="3"/>
+<pinref part="U1" gate="G$1" pin="5"/>
+<label x="176.53" y="48.514" size="1.27" layer="95" rot="R180" xref="yes"/>
+<wire x1="179.07" y1="48.514" x2="150.876" y2="48.514" width="0.1524" layer="91"/>
+<pinref part="JP6" gate="A" pin="1"/>
 </segment>
 </net>
@@
 </segment>
 </net>
+<net name="DATA_DISPLAY" class="0">
+<segment>
+<pinref part="U1" gate="G$1" pin="21"/>
+<label x="229.87" y="40.894" size="1.27" layer="95" xref="yes"/>
+<wire x1="226.06" y1="40.894" x2="254" y2="40.894" width="0.1524" layer="91"/>
+<pinref part="JP9" gate="A" pin="3"/>
+</segment>
+</net>
