File: IR_Station/eagle v3.0 corectare i2c pins/SolderingStation.sch (EAGLE design)
At the start: 104 parts, among them IC1 LM317, J1 JP4, J2 JP4, J3 JP4, J4 JP4, U1 MSP340G2443, U2 UPD166010, U3 MCP6V08, U4 UPD166010, U5 MCP6V08, U6 ADS1115IDGST

Commit message: 04.04.2018
Parts:
- removed JP13: (no value), adafruit:PINHD-1X1
- removed JP14, JP7: (no value), pinhead:PINHD-1X2
- removed JP9: (no value), pinhead:PINHD-1X9
- removed LED1: (no value), led:LEDCHIPLED_0603
- removed R19: 295, H_bridge_library:R1206
- added C15, C8: 1nF, adi_v1.2:C0805
- added D13: (no value), diode:DIODE-2AC|CASOT23
- added R25: 180R, adi_v1.2:R0805
- added R34: 0R, adi_v1.2:R0805
- added R35: 83R, adi_v1.2:R0805
- added R36: 295, H_bridge_library:R1206
- added U$12: (no value), Serghei IR station:COIL
- C2: value 10uF -> 2.4nF
- JP2: device pinhead:PINHD-1X5 -> pinhead:PINHD-1X2
- JP4: device adafruit:PINHD-1X1 -> pinhead:PINHD-2X9
- JP6: device pinhead:PINHD-1X6 -> pinhead:PINHD-2X10/90
- R16: value N/A -> 0R
- R23: value N/A -> 1K8
- R6: value 4K7 -> 15K
Connections:
- removed net 220V_DRIVER_UC: JP9.3, U1.21
- removed net DATA_DISPLAY: JP6.3, U1.5
- removed net ENCODER1_1: JP9.8, U1.16
- removed net ENCODER1_2: JP9.7, U1.17
- removed net ENCODER1_3: JP9.6, U1.18
- removed net ENCODER2_1: JP2.5, U1.10
- removed net ENCODER2_2: JP2.4, U1.11
- removed net ENCODER2_3: JP2.3, U1.12
- removed net ENCODER3_1: JP7.1, U1.27
- removed net ENCODER3_2: JP7.2, U1.26
- removed net ENCODER3_3: JP9.1, U1.23
- removed net LATCH_DISPLAY: JP9.5, U1.19
- removed net N$1: JP14.2, JP5.3
- removed net N$17: LED1.A, R19.2, R21.1
- new net +3V3_UC_LOCAL: C1.1, J1.1, J2.1, J3.1, J4.1, JP10.3, JP2.1, R18.2, R24.2, R32.2, U1.1
- new net 220V_PWM_LED_UC: JP4.17, R36.1
- new net 220V_PWM_UC: R36.2, U1.8
- new net 24V_PWM_LED_UC: JP4.3, R25.2
- new net BLANK_UC: JP4.4
- new net BUTTON1_UC: JP4.8, U1.18
- new net BUTTON2_UC: JP4.5, U1.12
- new net BUTTON3_UC: JP4.11, U1.5
- new net CLOCK_DISPLAY_UC: JP4.2
- new net DATA_DISPLAY_UC: JP4.1, U1.21
- new net ENCODER1_1_UC: JP4.16, U1.16
- new net ENCODER1_2_UC: JP4.14, U1.17
- new net ENCODER2_1_UC: JP4.9, U1.10
- new net ENCODER2_2_UC: JP4.7, U1.11
- new net ENCODER3_1_UC: JP4.15, U1.27
- new net ENCODER3_2_UC: JP4.13, U1.26
- new net FET_PWM_LED_UC: JP4.18, R35.1
- new net LATCH_DISPLAY_UC: JP4.6, U1.19
- new net N$28: D13.C, R35.2
- new net N$37: C8.1, U$12.P$2, U1.6
- new net N$39: C15.2, U$12.P$1, U1.7
- new net N$46: CLH1.IN, R34.1
- new net N$56: J1.4
- net +3V3_UC: now also JP2.2, JP4.10; no longer C1.1, J1.4, J2.4, J3.4, J4.4, JP10.3, JP13.1, R18.2, R24.2, R32.2, U1.1
- net 24V_CS_UC: no longer JP6.6
- net 24V_PWM: now also R34.2; no longer CLH1.IN
- net 24V_PWM_UC: now also R25.1, U1.9; no longer JP9.2, U1.22
- net CLOCK_DISPLAY: no longer JP9.9
- net FET_PWM1_UC: now also D13.A2; no longer JP2.2
- net FET_PWM2_UC: now also D13.A1; no longer JP2.1
- net GND: now also C15.1, C8.2, J2.4, J3.4, J4.4
- net GND_220V: no longer LED1.C
- net GND_UC: now also JP4.12; no longer J1.1, J2.1, J3.1, J4.1, JP4.1
- net N$15: now also R21.1; no longer R19.1
- net RX: no longer JP6.5
- net SCL: now also J1.3, J2.3, J3.3, J4.3, U1.22; no longer J1.2, J2.2, J3.2, J4.2, U1.9
- net SDA: now also J1.2, J2.2, J3.2, J4.2, U1.23; no longer J1.3, J2.3, J3.3, J4.3, U1.8
- net SPEAKER: now also JP5.3; no longer JP14.1
- net SPEAKER_UC: no longer JP9.4
- net TIP_TEMP1_UC: now also U$12.P$3; no longer JP6.2, U1.6
- net TIP_TEMP2_UC: now also U$12.P$4; no longer JP6.1, U1.7
- net TX: no longer JP6.4
Other:
- note added: "(20AMAX/K(15000) 2.5V)"
- note added: "2.5V(Ref msp430)/"
- note removed: "1.080V"
- note removed: "1.824V"
- note removed: "5mA"
- note removed: "6mA"
- note removed: "????"
- note removed: "ECU"
- moved on the sheet: C1, J1, J2, J3, J4, JP1, JP10, R18, R24, R32, U1
